Commit message: Update Parameters

File: src/guardian_description/urdf/robot_base.xacro (robot description, xacro)
@@ -13,6 +13,6 @@
     <xacro:property name="base_z_size" value="0.100" />
     <!-- Wheel Mounting Positions -->
-    <xacro:property name="wheelbase" value="0.400" />             <!-- x - Forward -->
-    <xacro:property name="track" value="0.350" />                 <!-- y - Side -->
+    <xacro:property name="wheelbase" value="0.400" />             <!-- the distance between the front and rear axles -->
+    <xacro:property name="track" value="0.350" />                 <!-- the distance between the left and right wheels -->
     <xacro:property name="wheel_vertical_offset" value="0.03" />
     <!-- Wheel Properties -->

File: src/guardian_description/urdf/ros2_control.xacro (robot description, xacro)
@@ -5,5 +5,5 @@
                sim_gazebo_classic:=^|false"
   >
-    <ros2_control name="${prefix}bot_ros2control" type="system">
+    <ros2_control name="${prefix}base_ros2control" type="system">
         <hardware>
           <xacro:if value="$(arg sim_gazebo_classic)">

Commit message: Update Simulation

File: src/guardian_description/urdf/robot_base.xacro (robot description, xacro)
@@ -22,5 +22,5 @@
     <link name="${prefix}base_link">
       <visual>
-        <origin xyz="0 0 ${base_z_size*3/4-0.01}" rpy="0 0 0" />
+        <origin xyz="0 0 ${base_z_size*2/4-0.01}" rpy="0 0 0" />
         <geometry>
           <box size="${base_x_size} ${base_y_size} ${base_z_size/2-0.02}"/>
@@ -28,5 +28,5 @@
       </visual>
       <collision>
-        <origin xyz="0 0 ${base_z_size*3/4-0.01}" rpy="0 0 0" />
+        <origin xyz="0 0 ${base_z_size*2/4-0.01}" rpy="0 0 0" />
         <geometry>
           <box size="${base_x_size} ${base_y_size} ${base_z_size/2-0.02}"/>

File: src/guardian_description/urdf/wheel.xacro (robot description, xacro)
@@ -11,5 +11,5 @@
         <origin xyz="0 0 0" rpy="0 0 0" />
         <geometry>
-          <mesh filename="package://guardian_description/meshes/wheel.dae" scale="0.4 0.4 0.4"/>
+          <mesh filename="package://guardian_description/meshes/wheel.dae" scale="0.3 0.3 0.3"/>
         </geometry>
       </visual>
