Commit message: Add manipulator ros2_control

File: src/guardian_description/urdf/manipulator.urdf.xacro (robot description, xacro)
@@ -1,11 +1,28 @@
 <?xml version="1.0"?>
-<robot xmlns:xacro="http://wiki.ros.org/xacro" name="r6bot">
+<robot xmlns:xacro="http://wiki.ros.org/xacro" name="guardian_manipulator">
+  <!-- paramters to be set from the launch file -->
+  <xacro:arg name="lower_limit" default="${str(-pi/2)}"/>
+  <xacro:arg name="upper_limit" default="${str(pi/2)}"/>
+  <xacro:arg name="sim_gazebo_classic" default="false"/>
+  <xacro:arg name="simulation_controllers" default=""/>
   <!-- Import r6bot macro -->
   <xacro:include filename="$(find guardian_description)/urdf/manipulator_macros.xacro"/>
   <!-- create link fixed to the "world" -->
   <link name="world"/>
-  <xacro:manipulator_description/>
-  <!-- Import r6bot ros2_control description -->
-  <!-- <xacro:include filename="$(find ros2_control_demo_example_7)/ros2_control/r6bot.ros2_control.xacro" />
-  <xacro:r6bot_ros2_control name="r6bot"/> -->
+  <xacro:manipulator_description
+    lower_joint_limit="$(arg lower_limit)"
+    upper_joint_limit="$(arg upper_limit)"/>
+  <!-- ros2_control -->
+  <xacro:include filename="$(find guardian_description)/ros2_control/manipulator.ros2_control.xacro"/>
+  <xacro:guardian_manipulator_ros2_control
+    lower_joint_limit="$(arg lower_limit)"
+    upper_joint_limit="$(arg upper_limit)"
+    sim_gazebo_classic="$(arg sim_gazebo_classic)"/>
+  <xacro:if value="$(arg sim_gazebo_classic)">
+    <gazebo>
+      <plugin filename="libgazebo_ros2_control.so" name="gazebo_ros2_control">
+        <parameters>$(arg simulation_controllers)</parameters>
+      </plugin>
+    </gazebo>
+  </xacro:if>
 </robot>

File: src/guardian_description/urdf/manipulator_macros.xacro (robot description, xacro)
@@ -1,10 +1,10 @@
 <?xml version="1.0"?>
 <robot xmlns:xacro="http://www.ros.org/wiki/xacro">
-  <xacro:macro name="manipulator_description">
+  <xacro:macro name="manipulator_description" params="
+               lower_joint_limit:=^|${-pi/2}
+               upper_joint_limit:=^|${pi/2}"
+  >
   <!-- helper macro -->
   <xacro:include filename="$(find guardian_description)/urdf/utils/create_link.xacro"/>
-  <!-- Joints Limits -->
-  <xacro:property name="lower_limit" value="${-pi/2}" />
-  <xacro:property name="upper_limit" value="${pi/2}" />
   <!-- Links -->
   <xacro:property name="link0_len" value="0.0793" />
@@ -80,5 +80,5 @@
     <origin xyz="0 0 ${link0_len}" rpy="0 0 0"/>
     <axis xyz="0 0 1"/>
-    <limit effort="1000.0" lower="${lower_limit}" upper="${upper_limit}" velocity="2.5"/>
+    <limit effort="1000.0" lower="${lower_joint_limit}" upper="${upper_joint_limit}" velocity="2.5"/>
   </joint>
   <joint name="joint_2" type="revolute">
@@ -87,5 +87,5 @@
     <origin xyz="0 0 ${link1_len}" rpy="0 0 0"/>
     <axis xyz="0 1 0"/>
-    <limit effort="1000.0" lower="${lower_limit}" upper="${upper_limit}" velocity="2.5"/>
+    <limit effort="1000.0" lower="${lower_joint_limit}" upper="${upper_joint_limit}" velocity="2.5"/>
   </joint>
   <joint name="joint_3" type="revolute">
@@ -94,5 +94,5 @@
     <origin xyz="0 0 ${link2_len}" rpy="0 0 0"/>
     <axis xyz="0 1 0"/>
-    <limit effort="1000.0" lower="${lower_limit}" upper="${upper_limit}" velocity="2.5"/>
+    <limit effort="1000.0" lower="${lower_joint_limit}" upper="${upper_joint_limit}" velocity="2.5"/>
   </joint>
   <joint name="joint_4" type="revolute">
@@ -101,5 +101,5 @@
     <origin xyz="0 0 ${link3_len}" rpy="0 0 0"/>
     <axis xyz="0 1 0"/>
-    <limit effort="1000.0" lower="${lower_limit}" upper="${upper_limit}" velocity="2.5"/>
+    <limit effort="1000.0" lower="${lower_joint_limit}" upper="${upper_joint_limit}" velocity="2.5"/>
   </joint>
   <joint name="joint_5" type="revolute">
@@ -108,5 +108,5 @@
     <origin xyz="0 0 ${link4_len}" rpy="0 0 0"/>
     <axis xyz="0 0 1"/>
-    <limit effort="1000.0" lower="${lower_limit}" upper="${upper_limit}" velocity="2.5"/>
+    <limit effort="1000.0" lower="${lower_joint_limit}" upper="${upper_joint_limit}" velocity="2.5"/>
   </joint>
 </xacro:macro>

File: src/guardian_description/urdf/robot.urdf.xacro (robot description, xacro)
@@ -7,5 +7,5 @@
   <!-- Included URDF/XACRO Files -->
   <xacro:include filename="$(find guardian_description)/urdf/robot_base.xacro"/>
-  <xacro:include filename="$(find guardian_description)/urdf/ros2_control.xacro"/>
+  <xacro:include filename="$(find guardian_description)/ros2_control/base.ros2_control.xacro"/>
   <!-- Load Base -->
   <xacro:guardian_base prefix="$(arg prefix)"/>
@@ -23,3 +23,4 @@
     </gazebo>
   </xacro:if>
+  <!-- Load Manipulator -->
 </robot>
