Commit message: ....

File: src/guardian_description/urdf/core/manipulator_macros.xacro (robot description, xacro)
@@ -93,5 +93,5 @@
     <child link="link_2"/>
     <origin xyz="0 0 ${link1_len}" rpy="0 0 0"/>
-    <axis xyz="0 1 0"/>
+    <axis xyz="0 -1 0"/>
     <limit effort="1000.0" lower="${lower_joint_limit}" upper="${upper_joint_limit}" velocity="2.5"/>
   </joint>

File: src/guardian_description/urdf/robot.urdf.xacro (robot description, xacro)
@@ -7,5 +7,4 @@
   <xacro:arg name="simulation_controllers" default="" />
   <!--Manipulator Args -->
-  <!-- <xacro:arg name="lower_limit" default="${str(-pi/2)}"/> -->
   <xacro:arg name="lower_limit" default="0.0"/>
   <xacro:arg name="upper_limit" default="${str(pi)}"/>

Commit message: ...

File: src/guardian_description/urdf/core/manipulator_macros.xacro (robot description, xacro)
@@ -92,6 +92,6 @@
     <parent link="link_1"/>
     <child link="link_2"/>
-    <origin xyz="0 0 ${link1_len}" rpy="0 0 0"/>
-    <axis xyz="0 -1 0"/>
+    <origin xyz="0 0 ${link1_len}" rpy="0 ${pi} 0"/>
+    <axis xyz="0 1 0"/>
     <limit effort="1000.0" lower="${lower_joint_limit}" upper="${upper_joint_limit}" velocity="2.5"/>
   </joint>

Commit message: ...

File: src/guardian_description/urdf/core/manipulator_macros.xacro (robot description, xacro)
@@ -93,5 +93,5 @@
     <child link="link_2"/>
     <origin xyz="0 0 ${link1_len}" rpy="0 ${pi} 0"/>
-    <axis xyz="0 1 0"/>
+    <axis xyz="0 -1 0"/>
     <limit effort="1000.0" lower="${lower_joint_limit}" upper="${upper_joint_limit}" velocity="2.5"/>
   </joint>

Commit message: Add moveit config

File: src/guardian_description/urdf/core/manipulator_macros.xacro (robot description, xacro)
@@ -94,5 +94,5 @@
     <origin xyz="0 0 ${link1_len}" rpy="0 ${pi} 0"/>
     <axis xyz="0 -1 0"/>
-    <limit effort="1000.0" lower="${upper_joint_limit}" upper="${lower_joint_limit}" velocity="2.5"/>
+    <limit effort="1000.0" lower="${lower_joint_limit}" upper="${upper_joint_limit}" velocity="2.5"/>
   </joint>
   <joint name="joint_3" type="revolute">
