Commit message: Finishing simulation

File: src/guardian_description/ros2_control/manipulator.ros2_control.xacro (robot description, xacro)
@@ -36,5 +36,5 @@
         </command_interface>
         <state_interface name="position">
-          <param name="initial_value">-0.450</param>
+          <param name="initial_value">-0.382</param>
         </state_interface>
         <state_interface name="velocity"/>
@@ -50,5 +50,5 @@
         </command_interface>
         <state_interface name="position">
-          <param name="initial_value">{pi/2}</param>
+          <param name="initial_value">1.36</param>
         </state_interface>
         <state_interface name="velocity"/>
@@ -64,5 +64,5 @@
         </command_interface>
         <state_interface name="position">
-          <param name="initial_value">1.04</param>
+          <param name="initial_value">0.858</param>
         </state_interface>
         <state_interface name="velocity"/>

File: src/guardian_description/urdf/core/manipulator_macros.xacro (robot description, xacro)
@@ -3,8 +3,9 @@
   <xacro:macro name="manipulator_description" params="
                lower_joint_limit:=^|${-pi/2}
-               upper_joint_limit:=^|${pi/2}"
+               upper_joint_limit:=^|${pi/2}
+               fix_link_to_robot_base:=^|false"
   >
   <!-- helper macro -->
-  <xacro:include filename="$(find guardian_description)/urdf/utils/create_link.xacro"/>
+  <xacro:include filename="$(find guardian_description)/urdf/core/create_link.xacro"/>
   <!-- Links -->
   <xacro:property name="link0_len" value="0.0793" />
@@ -15,5 +16,5 @@
   <xacro:property name="link5_len" value="0.1143" />
   <xacro:create_link
-    link_name="base_link"
+    link_name="manipulator_base_link"
     color="green"
     xyz_offset="0 0 ${link0_len/2}"
@@ -70,11 +71,17 @@
   <!-- Joints -->
   <joint name="base_joint" type="fixed">
-    <parent link="world"/>
-    <child link="base_link"/>
-    <origin xyz="0 0 0" rpy="0 0 0"/>
+    <xacro:if value="${fix_link_to_robot_base}">
+      <parent link="base_link"/>
+      <origin xyz="0 0 0.05" rpy="0 0 0"/>
+    </xacro:if>
+    <xacro:unless value="${fix_link_to_robot_base}">
+      <parent link="world"/>
+      <origin xyz="0 0 0" rpy="0 0 0"/>
+    </xacro:unless>
+    <child link="manipulator_base_link"/>
     <axis xyz="0 0 1"/>
   </joint>
   <joint name="joint_1" type="revolute">
-    <parent link="base_link"/>
+    <parent link="manipulator_base_link"/>
     <child link="link_1"/>
     <origin xyz="0 0 ${link0_len}" rpy="0 0 0"/>

File: src/guardian_description/urdf/core/robot_base.xacro (robot description, xacro)
@@ -6,5 +6,5 @@
   <xacro:property name="M_PI" value="3.14159"/>
   <!-- Included URDF/XACRO Files -->
-  <xacro:include filename="$(find guardian_description)/urdf/wheel.xacro" />
+  <xacro:include filename="$(find guardian_description)/urdf/core/wheel.xacro" />
   <xacro:macro name="guardian_base" params="prefix">
     <!-- Base Size -->

File: src/guardian_description/urdf/robot.urdf.xacro (robot description, xacro)
@@ -3,24 +3,46 @@
   <!-- paramters to be set from the launch file -->
   <xacro:arg name="prefix" default="" />
+  <xacro:arg name="use_robot_base" default="true" />
   <xacro:arg name="sim_gazebo_classic" default="false" />
   <xacro:arg name="simulation_controllers" default="" />
-  <!-- Included URDF/XACRO Files -->
-  <xacro:include filename="$(find guardian_description)/urdf/robot_base.xacro"/>
-  <xacro:include filename="$(find guardian_description)/ros2_control/base.ros2_control.xacro"/>
-  <!-- Load Base -->
-  <xacro:guardian_base prefix="$(arg prefix)"/>
-  <xacro:guardian_base_ros2_control
-    prefix="$(arg prefix)"
+  <!--Manipulator Args -->
+  <xacro:arg name="lower_limit" default="${str(-pi/2)}"/>
+  <xacro:arg name="upper_limit" default="${str(pi/2)}"/>
+  <!-- Robot Base -->
+  <xacro:if value="$(arg use_robot_base)">
+    <xacro:include filename="$(find guardian_description)/urdf/core/robot_base.xacro"/>
+    <xacro:include filename="$(find guardian_description)/ros2_control/base.ros2_control.xacro"/>
+    <xacro:guardian_base prefix="$(arg prefix)"/>
+    <xacro:guardian_base_ros2_control
+      prefix="$(arg prefix)"
+      sim_gazebo_classic="$(arg sim_gazebo_classic)"/>
+  <!-- Load Manipulator -->
+  <xacro:include filename="$(find guardian_description)/urdf/core/manipulator_macros.xacro"/>
+  <!-- create link fixed to the "world" -->
+  <xacro:unless value="$(arg use_robot_base)">
+    <link name="world"/>
+  </xacro:unless>
+  <xacro:manipulator_description
+    fix_link_to_robot_base="$(arg use_robot_base)"
+    lower_joint_limit="$(arg lower_limit)"
+    upper_joint_limit="$(arg upper_limit)"/>
+  <!-- ros2_control -->
+  <xacro:include filename="$(find guardian_description)/ros2_control/manipulator.ros2_control.xacro"/>
+  <xacro:guardian_manipulator_ros2_control
+    lower_joint_limit="$(arg lower_limit)"
+    upper_joint_limit="$(arg upper_limit)"
     sim_gazebo_classic="$(arg sim_gazebo_classic)"/>
+  <!-- Gazebo Classic -->
   <xacro:if value="$(arg sim_gazebo_classic)">
-    <gazebo>
-      <plugin filename="libgazebo_ros2_control.so" name="gazebo_ros2_control">
-        <parameters>$(arg simulation_controllers)</parameters>
-        <ros>
-          <remapping>/base_controller/cmd_vel_unstamped:=/cmd_vel</remapping>
-        </ros>
-      </plugin>
-    </gazebo>
+    <xacro:include filename="$(find guardian_simulation)/urdf/gazebo.urdf.xacro"/>
+      <gazebo>
+        <plugin filename="libgazebo_ros2_control.so" name="gazebo_ros2_control">
+          <parameters>$(arg simulation_controllers)</parameters>
+          <ros>
+            <remapping>/base_controller/cmd_vel_unstamped:=/cmd_vel</remapping>
+          </ros>
+        </plugin>
+      </gazebo>
+    </xacro:if>
   </xacro:if>
-  <!-- Load Manipulator -->
 </robot>

Commit message: Integrate URDF

File: src/guardian_description/ros2_control/manipulator.ros2_control.xacro (robot description, xacro)
@@ -6,4 +6,9 @@
                sim_gazebo_classic:=^|false"
   >
+  <xacro:property name="j1_init" value="0.0"/>
+  <xacro:property name="j2_init" value="-0.382"/>
+  <xacro:property name="j3_init" value="1.36"/>
+  <xacro:property name="j4_init" value="0.858"/>
+  <xacro:property name="j5_init" value="0.0"/>
     <ros2_control name="manipulator_ros2control" type="system">
       <hardware>
@@ -13,5 +18,18 @@
         <!-- Physical HW -->
         <xacro:unless value="$(arg sim_gazebo_classic)">
-          <plugin>gazebo_ros2_control/GazeboSystem</plugin>
+          <plugin>guardian/Pca9685SystemHardware</plugin>
+          <param name="pca_frequency">50.0</param>
+          <param name="jt_lower_limit">{lower_joint_limit}</param>
+          <param name="jt_upper_limit">{upper_joint_limit}</param>
+          <param name="joint_1__channel">9</param>
+          <param name="joint_2__channel">10</param>
+          <param name="joint_3__channel">11</param>
+          <param name="joint_4__channel">12</param>
+          <param name="joint_5__channel">13</param>
+          <param name="joint_1__init_position">{j1_init}</param>
+          <param name="joint_2__init_position">{j2_init}</param>
+          <param name="joint_3__init_position">{j3_init}</param>
+          <param name="joint_4__init_position">{j4_init}</param>
+          <param name="joint_5__init_position">{j5_init}</param>
         </xacro:unless>
       </hardware>
@@ -21,12 +39,7 @@
           <param name="max">{upper_joint_limit}</param>
         </command_interface>
-        <command_interface name="velocity">
-          <param name="min">-3.15</param>
-          <param name="max">3.15</param>
-        </command_interface>
         <state_interface name="position">
-          <param name="initial_value">0.0</param>
+          <param name="initial_value">{j1_init}</param>
         </state_interface>
-        <state_interface name="velocity"/>
       </joint>
       <joint name="joint_2">
@@ -35,12 +48,7 @@
           <param name="max">{upper_joint_limit}</param>
         </command_interface>
-        <command_interface name="velocity">
-          <param name="min">-3.15</param>
-          <param name="max">3.15</param>
-        </command_interface>
         <state_interface name="position">
-          <param name="initial_value">-0.382</param>
+          <param name="initial_value">{j2_init}</param>
         </state_interface>
-        <state_interface name="velocity"/>
       </joint>
       <joint name="joint_3">
@@ -49,12 +57,7 @@
           <param name="max">{upper_joint_limit}</param>
         </command_interface>
-        <command_interface name="velocity">
-          <param name="min">-3.15</param>
-          <param name="max">3.15</param>
-        </command_interface>
         <state_interface name="position">
-          <param name="initial_value">1.36</param>
+          <param name="initial_value">{j3_init}</param>
         </state_interface>
-        <state_interface name="velocity"/>
       </joint>
       <joint name="joint_4">
@@ -63,12 +66,7 @@
           <param name="max">{upper_joint_limit}</param>
         </command_interface>
-        <command_interface name="velocity">
-          <param name="min">-3.2</param>
-          <param name="max">3.2</param>
-        </command_interface>
         <state_interface name="position">
-          <param name="initial_value">0.858</param>
+          <param name="initial_value">{j4_init}</param>
         </state_interface>
-        <state_interface name="velocity"/>
       </joint>
       <joint name="joint_5">
@@ -77,12 +75,7 @@
           <param name="max">{upper_joint_limit}</param>
         </command_interface>
-        <command_interface name="velocity">
-          <param name="min">-3.2</param>
-          <param name="max">3.2</param>
-        </command_interface>
         <state_interface name="position">
-          <param name="initial_value">0.0</param>
+          <param name="initial_value">{j5_init}</param>
         </state_interface>
-        <state_interface name="velocity"/>
       </joint>
     </ros2_control>

Commit message: Add bringup

File: src/guardian_description/ros2_control/manipulator.ros2_control.xacro (robot description, xacro)
@@ -7,7 +7,10 @@
   >
   <xacro:property name="j1_init" value="0.0"/>
-  <xacro:property name="j2_init" value="-0.382"/>
+  <xacro:property name="j2_init" value="0.0"/>
+  <xacro:property name="j3_init" value="0.0"/>
+  <xacro:property name="j4_init" value="0.0"/>
+  <!-- <xacro:property name="j2_init" value="-0.382"/>
   <xacro:property name="j3_init" value="1.36"/>
-  <xacro:property name="j4_init" value="0.858"/>
+  <xacro:property name="j4_init" value="0.858"/> -->
   <xacro:property name="j5_init" value="0.0"/>
     <ros2_control name="manipulator_ros2control" type="system">
@@ -22,9 +25,9 @@
           <param name="jt_lower_limit">{lower_joint_limit}</param>
           <param name="jt_upper_limit">{upper_joint_limit}</param>
-          <param name="joint_1__channel">9</param>
-          <param name="joint_2__channel">10</param>
-          <param name="joint_3__channel">11</param>
-          <param name="joint_4__channel">12</param>
-          <param name="joint_5__channel">13</param>
+          <param name="joint_1__channel">0</param>
+          <param name="joint_2__channel">4</param>
+          <param name="joint_3__channel">12</param>
+          <param name="joint_4__channel">7</param>
+          <param name="joint_5__channel">5</param>
           <param name="joint_1__init_position">{j1_init}</param>
           <param name="joint_2__init_position">{j2_init}</param>

File: src/guardian_description/urdf/robot.urdf.xacro (robot description, xacro)
@@ -7,6 +7,7 @@
   <xacro:arg name="simulation_controllers" default="" />
   <!--Manipulator Args -->
-  <xacro:arg name="lower_limit" default="${str(-pi/2)}"/>
-  <xacro:arg name="upper_limit" default="${str(pi/2)}"/>
+  <!-- <xacro:arg name="lower_limit" default="${str(-pi/2)}"/> -->
+  <xacro:arg name="lower_limit" default="0.0"/>
+  <xacro:arg name="upper_limit" default="${str(pi}"/>
   <!-- Robot Base -->
   <xacro:if value="$(arg use_robot_base)">

Commit message: ...

File: src/guardian_description/ros2_control/manipulator.ros2_control.xacro (robot description, xacro)
@@ -7,10 +7,7 @@
   >
   <xacro:property name="j1_init" value="0.0"/>
-  <xacro:property name="j2_init" value="0.0"/>
-  <xacro:property name="j3_init" value="0.0"/>
-  <xacro:property name="j4_init" value="0.0"/>
-  <!-- <xacro:property name="j2_init" value="-0.382"/>
+  <xacro:property name="j2_init" value="-0.382"/>
   <xacro:property name="j3_init" value="1.36"/>
-  <xacro:property name="j4_init" value="0.858"/> -->
+  <xacro:property name="j4_init" value="0.858"/>
   <xacro:property name="j5_init" value="0.0"/>
     <ros2_control name="manipulator_ros2control" type="system">

Commit message: ...

File: src/guardian_description/ros2_control/manipulator.ros2_control.xacro (robot description, xacro)
@@ -7,7 +7,7 @@
   >
   <xacro:property name="j1_init" value="0.0"/>
-  <xacro:property name="j2_init" value="-0.382"/>
-  <xacro:property name="j3_init" value="1.36"/>
-  <xacro:property name="j4_init" value="0.858"/>
+  <xacro:property name="j2_init" value="3.1"/>
+  <xacro:property name="j3_init" value="0.0"/>
+  <xacro:property name="j4_init" value="0.0"/>
   <xacro:property name="j5_init" value="0.0"/>
     <ros2_control name="manipulator_ros2control" type="system">

Commit message: ...

File: src/guardian_description/ros2_control/manipulator.ros2_control.xacro (robot description, xacro)
@@ -20,6 +20,6 @@
           <plugin>guardian/Pca9685SystemHardware</plugin>
           <param name="pca_frequency">50.0</param>
-          <param name="jt_lower_limit">{lower_joint_limit}</param>
-          <param name="jt_upper_limit">{upper_joint_limit}</param>
+          <param name="jt_lower_limit">${lower_joint_limit}</param>
+          <param name="jt_upper_limit">${upper_joint_limit}</param>
           <param name="joint_1__channel">0</param>
           <param name="joint_2__channel">4</param>
@@ -27,54 +27,54 @@
           <param name="joint_4__channel">5</param>
           <param name="joint_5__channel">7</param>
-          <param name="joint_1__init_position">{j1_init}</param>
-          <param name="joint_2__init_position">{j2_init}</param>
-          <param name="joint_3__init_position">{j3_init}</param>
-          <param name="joint_4__init_position">{j4_init}</param>
-          <param name="joint_5__init_position">{j5_init}</param>
+          <param name="joint_1__init_position">${j1_init}</param>
+          <param name="joint_2__init_position">${j2_init}</param>
+          <param name="joint_3__init_position">${j3_init}</param>
+          <param name="joint_4__init_position">${j4_init}</param>
+          <param name="joint_5__init_position">${j5_init}</param>
         </xacro:unless>
       </hardware>
       <joint name="joint_1">
         <command_interface name="position">
-          <param name="min">{lower_joint_limit}</param>
-          <param name="max">{upper_joint_limit}</param>
+          <param name="min">${lower_joint_limit}</param>
+          <param name="max">${upper_joint_limit}</param>
         </command_interface>
         <state_interface name="position">
-          <param name="initial_value">{j1_init}</param>
+          <param name="initial_value">${j1_init}</param>
         </state_interface>
       </joint>
       <joint name="joint_2">
         <command_interface name="position">
-          <param name="min">{lower_joint_limit}</param>
-          <param name="max">{upper_joint_limit}</param>
+          <param name="min">${lower_joint_limit}</param>
+          <param name="max">${upper_joint_limit}</param>
         </command_interface>
         <state_interface name="position">
-          <param name="initial_value">{j2_init}</param>
+          <param name="initial_value">${j2_init}</param>
         </state_interface>
       </joint>
       <joint name="joint_3">
         <command_interface name="position">
-          <param name="min">{lower_joint_limit}</param>
-          <param name="max">{upper_joint_limit}</param>
+          <param name="min">${lower_joint_limit}</param>
+          <param name="max">${upper_joint_limit}</param>
         </command_interface>
         <state_interface name="position">
-          <param name="initial_value">{j3_init}</param>
+          <param name="initial_value">${j3_init}</param>
         </state_interface>
       </joint>
       <joint name="joint_4">
         <command_interface name="position">
-          <param name="min">{lower_joint_limit}</param>
-          <param name="max">{upper_joint_limit}</param>
+          <param name="min">${lower_joint_limit}</param>
+          <param name="max">${upper_joint_limit}</param>
         </command_interface>
         <state_interface name="position">
-          <param name="initial_value">{j4_init}</param>
+          <param name="initial_value">${j4_init}</param>
         </state_interface>
       </joint>
       <joint name="joint_5">
         <command_interface name="position">
-          <param name="min">{lower_joint_limit}</param>
-          <param name="max">{upper_joint_limit}</param>
+          <param name="min">${lower_joint_limit}</param>
+          <param name="max">${upper_joint_limit}</param>
         </command_interface>
         <state_interface name="position">
-          <param name="initial_value">{j5_init}</param>
+          <param name="initial_value">${j5_init}</param>
         </state_interface>
       </joint>

File: src/guardian_description/urdf/core/manipulator_macros.xacro (robot description, xacro)
@@ -94,5 +94,5 @@
     <origin xyz="0 0 ${link1_len}" rpy="0 ${pi} 0"/>
     <axis xyz="0 -1 0"/>
-    <limit effort="1000.0" lower="${lower_joint_limit}" upper="${upper_joint_limit}" velocity="2.5"/>
+    <limit effort="1000.0" lower="${upper_joint_limit}" upper="${lower_joint_limit}" velocity="2.5"/>
   </joint>
   <joint name="joint_3" type="revolute">

Commit message: ...

File: src/guardian_description/ros2_control/manipulator.ros2_control.xacro (robot description, xacro)
@@ -27,4 +27,5 @@
           <param name="joint_4__channel">5</param>
           <param name="joint_5__channel">7</param>
+          <param name="joint_6__channel">14</param>
           <param name="joint_1__init_position">${j1_init}</param>
           <param name="joint_2__init_position">${j2_init}</param>
@@ -79,4 +80,8 @@
         </state_interface>
       </joint>
+      <joint name="joint_6">
+        <command_interface name="position"/>
+        <state_interface name="position"/>
+      </joint>
     </ros2_control>
   </xacro:macro>

File: src/guardian_description/urdf/core/manipulator_macros.xacro (robot description, xacro)
@@ -14,5 +14,6 @@
   <xacro:property name="link3_len" value="0.18415" />
   <xacro:property name="link4_len" value="0.0635" />
-  <xacro:property name="link5_len" value="0.1143" />
+  <xacro:property name="link5_len" value="0.10" />
+  <xacro:property name="link6_len" value="0.05" />
   <xacro:create_link
     link_name="manipulator_base_link"
@@ -69,4 +70,13 @@
     y="0.035"
   />
+  <xacro:create_link
+    link_name="link_6"
+    color="blue"
+    xyz_offset="0 0 ${link6_len/2}"
+    rpy_offset="0 0 0"
+    z="${link6_len}"
+    x="0.0285"
+    y="0.035"
+  />
   <!-- Joints -->
   <joint name="base_joint" type="fixed">
@@ -117,4 +127,11 @@
     <limit effort="1000.0" lower="${lower_joint_limit}" upper="${upper_joint_limit}" velocity="2.5"/>
   </joint>
+  <joint name="joint_6" type="revolute">
+    <parent link="link_5"/>
+    <child link="link_6"/>
+    <origin xyz="0 0 ${link5_len}" rpy="0 0 0"/>
+    <axis xyz="0 0 1"/>
+    <limit effort="1000.0" lower="${lower_joint_limit}" upper="${upper_joint_limit}" velocity="2.5"/>
+  </joint>
 </xacro:macro>
 </robot>
