Commit message: ...

File: src/guardian_moveit_config/config/greenguardian.ros2_control.xacro (robot description, xacro)
@@ -43,4 +43,11 @@
                 <state_interface name="velocity"/>
             </joint>
+            <joint name="joint_6">
+                <command_interface name="position"/>
+                <state_interface name="position">
+                  <param name="initial_value">${initial_positions['joint_6']}</param>
+                </state_interface>
+                <state_interface name="velocity"/>
+            </joint>
         </ros2_control>
     </xacro:macro>
