Commit message: ...

File: src/guardian_description/urdf/extra/manipulator.urdf (robot description, URDF)
Before this commit: robot greenguardian, 7 links, 6 joints
Links:
- removed link world
- link manipulator_base_link: mass 1.0 -> None
Joints:
- removed joint base_joint

Commit message: ...

File: src/guardian_description/urdf/extra/manipulator.urdf (robot description, URDF)
Before this commit: robot greenguardian, 6 links, 5 joints
Links:
- added link link_6, mass 1.0; collision box size=0.0285 0.035 0.05; visual box size=0.0285 0.035 0.05
- added link world
- link link_5: geometry collision box size=0.0285 0.035 0.1; visual box size=0.0285 0.035 0.1
- link manipulator_base_link: mass None -> 1.0
Joints:
- added joint base_joint: type fixed, parent world, child manipulator_base_link, origin xyz=0 0 0 rpy=0 0 0, axis 0 0 1
- added joint joint_6: type revolute, parent link_5, child link_6, origin xyz=0 0 0.1 rpy=0 0 0, axis 0 0 1, limit lower=0.0 upper=3.141592653589793 effort=1000.0 velocity=2.5
- joint joint_2: limit lower=1.57 upper=3.141592653589793 effort=1000.0 velocity=2.5 -> lower=0.0 upper=3.141592653589793 effort=1000.0 velocity=2.5

Commit message: Add moveit

File: src/guardian_description/urdf/extra/manipulator.urdf (robot description, URDF)
Before this commit: robot greenguardian, 8 links, 7 joints
Joints:
- joint joint_1: limit lower=0.0 upper=3.141592653589793 effort=1000.0 velocity=2.5 -> lower=0.0 upper=6.0 effort=1000.0 velocity=2.5
- joint joint_2: limit lower=0.0 upper=3.141592653589793 effort=1000.0 velocity=2.5 -> lower=0.0 upper=6.0 effort=1000.0 velocity=2.5
- joint joint_3: limit lower=0.0 upper=3.141592653589793 effort=1000.0 velocity=2.5 -> lower=0.0 upper=6.0 effort=1000.0 velocity=2.5
- joint joint_4: limit lower=0.0 upper=3.141592653589793 effort=1000.0 velocity=2.5 -> lower=0.0 upper=6.0 effort=1000.0 velocity=2.5
- joint joint_5: limit lower=0.0 upper=3.141592653589793 effort=1000.0 velocity=2.5 -> lower=0.0 upper=6.0 effort=1000.0 velocity=2.5
- joint joint_6: limit lower=0.0 upper=3.141592653589793 effort=1000.0 velocity=2.5 -> lower=0.0 upper=6.0 effort=1000.0 velocity=2.5
